File: amoeba-ulp.kicad_pcb (KiCad board)
At the start: 2 copper layers, 18.2 x 16.8 mm, 6 parts

Commit message: mini v2
Parts:
- D1: footprint Diode_SMD:D_SOD-323 -> Diode_SMD:D_SOD-123
- moved C 2.80 mm to (105.0, 101.3)
- moved C 2.64 mm to (105.3, 111.5)
- moved R 1.90 mm to (101.3, 106.4)
- moved R 1.89 mm to (112.9, 106.4)
- renumbered ULP1 to ULP2
Routing:
- net Column: track 19.5 -> 10.5 mm
- net Row: track 17.4 -> 12.9 mm
Other:
- board size 18.2 x 16.8 mm -> 14.2 x 12.8 mm
